Commit message: examen, practica 1 bien y jupiter

File: practica1_description/urdf/basic_link.urdf (robot description, URDF)
Before this commit: robot basic_link, 2 links, 1 joints
Links:
- added link link_2, mass 1.0; collision box size=0.1 0.1 0.4; visual box size=0.1 0.1 0.4
Joints:
- added joint link_1_to_link_2_joint: type revolute, parent link_1, child link_2, origin xyz=0.0 0.10 0.5 rpy=0 0 0, axis 0 1 0, limit lower=-1.57 upper=1.57 effort=1000 velocity=1
- joint base_link_to_link_1_joint: axis 1 0 0 -> 0 1 0; origin xyz=0.0 0.0 0.15 rpy=0 0 0 -> xyz=0.0 0.05 0.20 rpy=0 0 0
