Commit message: archivo scara.urdf.xacro corregido y funcional

File: examen_description/urdf/scara.urdf.xacro (robot description, xacro)
@@ -26,5 +26,5 @@
     <link name="link_1">
         <visual>
-            <origin xyz="0.25 0.0 0.0" rpy="0.0 0.0 0.0" />
+            <origin xyz="0.25 0.0 0.025" rpy="0.0 0.0 0.0" />
             <geometry>
                 <box size="0.5 0.05 0.05" />
@@ -35,5 +35,5 @@
         </visual>
         <collision>
-            <origin xyz="0.25 0.0 0.0" rpy="0.0 0.0 0.0" />
+            <origin xyz="0.25 0.0 0.025" rpy="0.0 0.0 0.0" />
             <geometry>
                 <box size="0.5 0.05 0.05" />
@@ -46,5 +46,5 @@
         </inertial>
     </link>
-    <joint name="base_link_to_link_1_joint" type="revolute">
+    <joint name="ink_1_joint" type="revolute">
         <parent link="base_link" />
         <child link="link_1" />
@@ -52,9 +52,9 @@
         <limit lower="-1.57" upper="1.57" velocity="1"
             effort="1000" />
-        <origin xyz="0.0 0.0 0.225" rpy="0 0 0" />
+        <origin xyz="0.0 0.0 0.2" rpy="0 0 0" />
     </joint>
     <link name="link_2">
         <visual>
-            <origin xyz="0.0 0.0 0.25" rpy="0.0 0.0 0.0" />
+            <origin xyz="0.25 0.0 0.025" rpy="0.0 0.0 0.0" />
             <geometry>
                 <box size="0.5 0.05 0.05" />
@@ -65,5 +65,5 @@
         </visual>
         <collision>
-            <origin xyz="0.0 0.0 0.25" rpy="0.0 0.0 0.0" />
+            <origin xyz="0.25 0.0 0.025" rpy="0.0 0.0 0.0" />
             <geometry>
                 <box size="0.5 0.05 0.05" />
@@ -82,9 +82,9 @@
         <limit lower="-1.57" upper="1.57" velocity="1"
             effort="1000" />
-        <origin xyz="0.0 0.0 0.20" rpy="0 0 0" />
+        <origin xyz="0.5 0.0 0.05" rpy="0 0 0" />
     </joint>
     <link name="link_3">
         <visual>
-            <origin xyz="0.0 0.0 0.25" rpy="0.0 0.0 0.0" />
+            <origin xyz="0.25 0.0 0.025" rpy="0.0 0.0 0.0" />
             <geometry>
                 <box size="0.5 0.05 0.05" />
@@ -95,5 +95,5 @@
         </visual>
         <collision>
-            <origin xyz="0.0 0.0 0.25" rpy="0.0 0.0 0.0" />
+            <origin xyz="0.25 0.0 0.025" rpy="0.0 0.0 0.0" />
             <geometry>
                 <box size="0.5 0.05 0.05" />
@@ -112,5 +112,5 @@
         <limit lower="-1.57" upper="1.57" velocity="1"
             effort="1000" />
-        <origin xyz="0.0 0.0 0.20" rpy="0 0 0" />
+        <origin xyz="0.5 0.0 0.05" rpy="0 0 0" />
     </joint>
 </robot>

Commit message: PKG examen_bringup -> simple_position_controller.launch.py y scara_simple_controller.xacr en examen_descriptiono

File: examen_description/urdf/scara.urdf.xacro (robot description, xacro)
@@ -3,4 +3,13 @@
 <!--<robot name="robot_scara">-->
 <!--Descripcion del robot scara-->
+    <!--Creando anclaje-->
+    <link name="world">
+    </link>
+    <joint name="world_joint" type="fixed">
+        <parent link="world" />
+        <child link="base_link" />
+        <axis xyz="0 0 0" />
+        <origin xyz="0.0 0.0 0.0" rpy="0 0 0" />
+    </joint>
     <link name="base_link">
         <visual>
@@ -83,9 +92,9 @@
         <limit lower="-1.57" upper="1.57" velocity="1"
             effort="1000" />
-        <origin xyz="0.5 0.0 0.05" rpy="0 0 0" />
+        <origin xyz="0.45 0.0 0.05" rpy="0 0 0" />
     </joint>
     <link name="link_3">
         <visual>
-            <origin xyz="0.25 0.0 0.025" rpy="0.0 0.0 0.0" />
+            <origin xyz="0.25 0.0 -0.025" rpy="0.0 0.0 0.0" />
             <geometry>
                 <box size="0.5 0.05 0.05" />
@@ -96,5 +105,5 @@
         </visual>
         <collision>
-            <origin xyz="0.25 0.0 0.025" rpy="0.0 0.0 0.0" />
+            <origin xyz="0.25 0.0 -0.025" rpy="0.0 0.0 0.0" />
             <geometry>
                 <box size="0.5 0.05 0.05" />
@@ -113,5 +122,12 @@
         <limit lower="-1.57" upper="1.57" velocity="1"
             effort="1000" />
-        <origin xyz="0.5 0.0 0.05" rpy="0 0 0" />
+        <origin xyz="0.45 0.0 0.0" rpy="0 0 0" />
+    </joint>
+    <link name="P">
+    </link>
+    <joint name="link_P_joint" type="fixed">
+        <parent link="link_3" />
+        <child link="P" />
+        <origin xyz="0.45 0.0 0.0" rpy="0 0 0" />
     </joint>
 </robot>

Commit message: Scara Jalando en Gazebo, correccion scara_basic_position_controller.xacro

File: examen_description/urdf/scara.urdf.xacro (robot description, xacro)
@@ -3,5 +3,5 @@
 <!--<robot name="robot_scara">-->
 <!--Descripcion del robot scara-->
-    <!--Creando anclaje-->
+    <!--Creando anclaje para Gazebo-->
     <link name="world">
     </link>
@@ -12,4 +12,5 @@
         <origin xyz="0.0 0.0 0.0" rpy="0 0 0" />
     </joint>
+    <!--Fin anclaje-->
     <link name="base_link">
         <visual>
@@ -92,5 +93,5 @@
         <limit lower="-1.57" upper="1.57" velocity="1"
             effort="1000" />
-        <origin xyz="0.45 0.0 0.05" rpy="0 0 0" />
+        <origin xyz="0.5 0.0 0.05" rpy="0 0 0" />
     </joint>
     <link name="link_3">
@@ -122,5 +123,5 @@
         <limit lower="-1.57" upper="1.57" velocity="1"
             effort="1000" />
-        <origin xyz="0.45 0.0 0.0" rpy="0 0 0" />
+        <origin xyz="0.5 0.0 0.0" rpy="0 0 0" />
     </joint>
     <link name="P">
@@ -129,5 +130,5 @@
         <parent link="link_3" />
         <child link="P" />
-        <origin xyz="0.45 0.0 0.0" rpy="0 0 0" />
+        <origin xyz="0.5 0.0 0.0" rpy="0 0 0" />
     </joint>
 </robot>

File: examen_description/urdf/scara_basic_position_controller.xacro (robot description, xacro)
@@ -2,7 +2,8 @@
 <robot name="robot_scara" xmlns:xacro="http://ros.org/wiki/xacro">
     <gazebo>
-        <plugin name="joint-state_publisher_controller" filename="libgazebo_ros_joint_state_publisher.so">
+        <plugin name="joint_state_publisher_controller" filename="libgazebo_ros_joint_state_publisher.so">
             <!--update rate Hz-->
             <update_rate>10</update_rate>
+            <joint_name>link_1_joint</joint_name>
             <joint_name>link_2_joint</joint_name>
             <joint_name>link_3_joint</joint_name>
